File: LED_Wled.sch (KiCad schematic (older format))
At the start: 18 parts, among them J1 SWD_PORT_SKEDD, J2 Screw_Terminal_01x02, J3 Screw_Terminal_01x03, Q1 BSS138, U1 ESP8266-12E_ESP-12E, U2 AMS1117-3.3, U3 AMS1117-5.0

Commit message: library fixes
Parts:
- J1: footprint userdvc:WR_WST_REDFIT_IDC_4Pin -> LED_Wled:WR_WST_REDFIT_IDC_4Pin; symbol userdvc:SWD_PORT_SKEDD -> LED_Wled:SWD_PORT_SKEDD
Changed lines of the file:
@@
 	3250 3800 3250 3750
 $Comp
-L userdvc:SWD_PORT_SKEDD J1
+L LED_Wled:SWD_PORT_SKEDD J1
 U 1 1 6183A836
 P 4150 2250
 F 0 "J1" V 4330 1962 50  0000 R CNN
 F 1 "SWD_PORT_SKEDD" V 4239 1962 50  0000 R CNN
-F 2 "userdvc:WR_WST_REDFIT_IDC_4Pin" H 4150 2250 50  0001 C CNN
+F 2 "LED_Wled:WR_WST_REDFIT_IDC_4Pin" H 4150 2250 50  0001 C CNN
 F 3 "https://www.we-online.com/catalog/datasheet/490107670412.pdf" H 4150 2250 50  0001 C CNN
 F 4 "U-1367961" V 4148 1962 50  0000 R CNN "SKU"
