File: LED_Wled.sch (KiCad schematic (older format))
At the start: 17 parts, among them J1 SWD_PORT_SKEDD, J2 Screw_Terminal_01x02, J3 Screw_Terminal_01x03, Q1 BSS138, U1 ESP8266-12E_ESP-12E

Commit message: updated to rev1.1
Parts:
- added C4: 100nF/50V, Capacitor_SMD:C_0805_2012Metric, symbol Device:C_Small
- added C5: 10uF/50V, Capacitor_SMD:C_1206_3216Metric, symbol Device:C_Small
- added NT1: Net-Tie_2, NetTie:NetTie-2_SMD_Pad2.0mm, symbol Device:Net-Tie_2
- added U3: LD1117DT33TR, Package_TO_SOT_SMD:TO-252-2, symbol Regulator_Linear:LM1117-3.3
- BOOT1: renamed from JP1; footprint Jumper:SolderJumper-2_P1.3mm_Open_RoundedPad1.0x1.5mm -> Connector_PinHeader_1.27mm:PinHeader_1x02_P1.27mm_Vertical; JLCSMT - -> (none); JLCSMT_PKG - -> (none); JLCSMT_Part - -> (none); MANUFACTURER - -> (none); MPN - -> (none); SKU - -> (none); SPR - -> (none)
- C1: renamed from C?; value 330uF/35V -> 180uF/35V; footprint Capacitor_SMD:CP_Elec_10x10.5 -> Capacitor_SMD:CP_Elec_10x12.5; JLCSMT C88796 -> C488000; JLCSMT_Part 35TZV330M10X10.5 -> PCV1V181MCL2GS; MANUFACTURER Rubycon -> Nichicon
- C2: renamed from C?; value CP_Small -> 470uF/35V; footprint (none) -> Capacitor_SMD:C_Elec_10x10.2; JLCSMT (none) -> C3350; JLCSMT_PKG (none) -> SMD-ECAP-10x10; JLCSMT_Part (none) -> RVT1V471M1010; MANUFACTURER (none) -> Honor Elec
- C3: renamed from C?; value C_Small -> 1uF/50V; footprint (none) -> Capacitor_SMD:C_1206_3216Metric; JLCSMT (none) -> C1848; JLCSMT_PKG (none) -> 1206; JLCSMT_Part (none) -> CL31B105KBHNNNE; MANUFACTURER (none) -> Samsung Electro-Mechanics
- D1: renamed from D?; value D_Schottky_Small -> SS32; footprint (none) -> Diode_SMD:D_SMC; JLCSMT (none) -> C65005; JLCSMT_PKG (none) -> SMC,DO-214AB; JLCSMT_Part (none) -> SS32; MANUFACTURER (none) -> MDD（Microdiode Electronics）
- J1: JLCSMT - -> (none); JLCSMT_PKG - -> (none); JLCSMT_Part - -> (none); MANUFACTURER - -> (none); MFR WURTH ELEKTRONIK -> WURTH ELEKTRONIK
- J2: footprint TerminalBlock_TE-Connectivity:TerminalBlock_TE_282834-2_1x02_P2.54mm_Horizontal -> TerminalBlock_MetzConnect:TerminalBlock_MetzConnect_Type086_RT03402HBLC_1x02_P3.81mm_Horizontal; JLCSMT - -> C69811; JLCSMT_PKG - -> CONN-TH_2P-P3.81_KF124-3.81-2P; JLCSMT_Part - -> WJ124-3.81-2P; MANUFACTURER - -> Ningbo Kangnex Elec; MPN 282834-2 -> 282834-2; SPR Lemona -> (none)
- J3: footprint TerminalBlock_TE-Connectivity:TerminalBlock_TE_282834-3_1x03_P2.54mm_Horizontal -> TerminalBlock_MetzConnect:TerminalBlock_MetzConnect_Type086_RT03403HBLC_1x03_P3.81mm_Horizontal; JLCSMT - -> C36780; JLCSMT_PKG - -> CONN-TH; JLCSMT_Part - -> WJ124-3.81-3P; MANUFACTURER - -> Ningbo Kangnex Elec
- L1: renamed from L?; value 47uH -> 68uH; footprint Inductor_SMD:L_Bourns_SRN6045TA -> Inductor_SMD:L_12x12mm_H8mm; JLCSMT C497841 -> C169377; JLCSMT_PKG IND-SMD -> SMD-12.5x12.5x8; JLCSMT_Part YNR6045-470M -> SWRB1207S-680MT; MANUFACTURER YJYCOIN -> Sunlord
- Q1: JLCSMT - -> C400505; JLCSMT_PKG - -> SOT-23-3; JLCSMT_Part - -> BSS138; MANUFACTURER - -> Yangzhou Yangjie Elec Tech
- R1, R2, R3, R4, R5: JLCSMT C17724 -> C17414; JLCSMT_Part 0805W8F510KT5E -> 0805W8F1002T5E; MPN - -> (none); SKU - -> (none); SPR - -> (none)
- U1: JLCSMT - -> C82891; JLCSMT_PKG - -> DFN-22_16.0x24.0x2.0P; JLCSMT_Part - -> ESP-12F(ESP8266MOD); MPN - -> (none); SKU - -> (none)
- U2: renamed from U?; JLCSMT C74193 -> C61063; JLCSMT_Part XL1509-3.3E1 -> XL1509-5.0E1
Connections:
- net labels added: GNDPWR
- wire segments 60 -> 77
- no-connect marks 13 -> 14
Other:
- moved on the sheet: C1, C2, C3, D1, J1, J2, J3, L1, Q1, R4, R5, U2

Commit message: finished rev1.1
Parts:
- removed J2: Screw_Terminal_01x02, TerminalBlock_MetzConnect:TerminalBlock_MetzConnect_Type086_RT03402HBLC_1x02_P3.81mm_Horizontal, symbol Connector:Screw_Terminal_01x02
- removed J3: Screw_Terminal_01x03, TerminalBlock_MetzConnect:TerminalBlock_MetzConnect_Type086_RT03403HBLC_1x03_P3.81mm_Horizontal, symbol Connector:Screw_Terminal_01x03
- added F1: Fuse_Small, Fuse:Fuse_1812_4532Metric, symbol Device:Fuse_Small
- added J2: KF141V-2.54-2P, userdvc:KF141V-2.54-2P, symbol userdvc:KF141V-2.54-2P
- added J3: KF141V-2.54-3P, userdvc:KF141V-2.54-3P, symbol userdvc:KF141V-2.54-3P
- C1: value 180uF/35V -> 180uF/63V; footprint Capacitor_SMD:CP_Elec_10x12.5 -> Capacitor_THT:C_Radial_D10.0mm_H16.0mm_P5.00mm; JLCSMT C488000 -> C106532; JLCSMT_PKG CAP-SMD -> Radial,10X16mm; JLCSMT_Part PCV1V181MCL2GS -> ERF1JM181G16OT; MANUFACTURER Nichicon -> AISHI(Aihua Group)
Connections:
- wire segments 77 -> 78
Other:
- note added: "LDO POWER +3.3V"
- note added: "SWITCHING POWER +5V\n"
- moved on the sheet: C1, C2, C3, C4, C5, D1, L1, U2
