File: LED_Wled.kicad_pcb (KiCad board)
At the start: 2 copper layers, 100 x 97.5 mm, 125 parts, among them J1 SWD_PORT_SKEDD, J2 Screw_Terminal_01x02, J3 Screw_Terminal_01x03, Q1 BSS138, U1 ESP8266-12E_ESP-12E, U2 AMS1117-3.3, U3 AMS1117-5.0

Commit message: rev1.0 release
Parts:
- added G***: LOGO, LED_Wled:es, B.Cu at (98.5, 134.5)
- added G***: LOGO, LED_Wled:es, B.Cu at (98.5, 106.5)
- added G***: LOGO, LED_Wled:es, B.Cu at (121.5, 133.5)
- added G***: LOGO, LED_Wled:es, B.Cu at (121.5, 105.5)
- added G***: LOGO, LED_Wled:es, B.Cu at (121.5, 77.5)
- added G***: LOGO, LED_Wled:es, B.Cu at (98.5, 78.5)
Other:
- board text added: "remote-led-project 2021-11-04 rev1.0"

Commit message: rev1.0_PROD
Other:
- board text added: "For use with ARGB LED-strip MAX INPUT: +13V"
Changed lines of the file:
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@@
   (general
     (thickness 1.6)
-    (drawings 142)
+    (drawings 148)
     (tracks 606)
     (zones 0)
@@
     (tags "CMS SOT")
     (attr smd)
-    (fp_text reference U3 (at 0 -4.5 90) (layer F.SilkS)
+    (fp_text reference U3 (at 0 -4.1 90) (layer F.SilkS)
       (effects (font (size 1 1) (thickness 0.15)))
     )
@@
     (tags "CMS SOT")
     (attr smd)
-    (fp_text reference U3 (at 0 -4.5 90) (layer F.SilkS)
+    (fp_text reference U3 (at 0 -4.1 90) (layer F.SilkS)
       (effects (font (size 1 1) (thickness 0.15)))
     )
@@
     (tags "CMS SOT")
     (attr smd)
-    (fp_text reference U3 (at 0 -4.5 90) (layer F.SilkS)
+    (fp_text reference U3 (at 0 -4.1 90) (layer F.SilkS)
       (effects (font (size 1 1) (thickness 0.15)))
     )
@@
     (tags "CMS SOT")
     (attr smd)
-    (fp_text reference U3 (at 0 -4.5 90) (layer F.SilkS)
+    (fp_text reference U3 (at 0 -4.1 90) (layer F.SilkS)
       (effects (font (size 1 1) (thickness 0.15)))
     )
@@
     (tags "CMS SOT")
     (attr smd)
-    (fp_text reference U3 (at 0 -4.5 90) (layer F.SilkS)
+    (fp_text reference U3 (at 0 -4.1 90) (layer F.SilkS)
       (effects (font (size 1 1) (thickness 0.15)))
     )
@@
     (tags "CMS SOT")
     (attr smd)
-    (fp_text reference U3 (at 0 -4.5 90) (layer F.SilkS)
+    (fp_text reference U3 (at 0 -4.1 270) (layer F.SilkS)
       (effects (font (size 1 1) (thickness 0.15)))
     )
@@
     )
   )
+  (gr_text "For use with\nARGB LED-strip\nMAX INPUT: +13V" (at 141 69 180) (layer B.SilkS)
+    (effects (font (size 1.5 1.5) (thickness 0.3)) (justify mirror))
+  )
+  (gr_text "For use with\nARGB LED-strip\nMAX INPUT: +13V" (at 141 97 180) (layer B.SilkS)
+    (effects (font (size 1.5 1.5) (thickness 0.3)) (justify mirror))
+  )
+  (gr_text "For use with\nARGB LED-strip\nMAX INPUT: +13V" (at 141 125 180) (layer B.SilkS)
+    (effects (font (size 1.5 1.5) (thickness 0.3)) (justify mirror))
+  )
+  (gr_text "For use with\nARGB LED-strip\nMAX INPUT: +13V" (at 79 143) (layer B.SilkS)
+    (effects (font (size 1.5 1.5) (thickness 0.3)) (justify mirror))
+  )
+  (gr_text "For use with\nARGB LED-strip\nMAX INPUT: +13V" (at 79 115) (layer B.SilkS)
+    (effects (font (size 1.5 1.5) (thickness 0.3)) (justify mirror))
+  )
+  (gr_text "For use with\nARGB LED-strip\nMAX INPUT: +13V" (at 79 87) (layer B.SilkS)
+    (effects (font (size 1.5 1.5) (thickness 0.3)) (justify mirror))
+  )
   (gr_text "remote-led-project\n2021-11-04 rev1.0" (at 128 131.5 90) (layer B.SilkS)
